Commit message: test(export,ci): MuJoCo checks every site pose against our FK (plans/frames-and-sites step 3)
The risk this plan carries is that a `<site>` we write is not where we say
it is. This retires it the way M3 retired it for joints (ADR-0004 §2):
`<name>.fk.json` now carries `sites: {name: {pos, quat}}` beside `links` per
sample — `world(parent) ∘ frame.pose` from the same FK pass — and
`test_mjcf_load.py` sets each configuration, runs `mj_forward` and compares
`data.site(name)` (its `xmat` converted with `mju_mat2Quat`, since MuJoCo
has no `site_xquat`) to 1e-6. A site the samples name and the model lacks
is a failure, not a skip: that is exactly what a dropped `<site>` looks
like.

The arm fixture carries both routes now. `write_arm_sample` gives
`arm.riggen` a `tcp` 80 mm past the forearm and a `camera_mount` turned
onto the plinth's +X face, and the hand-written `arm.urdf` gains the two
massless dummy links riggen would write for them. So the existing `mujoco`
job proves the `.riggen` route through the sites and the URDF route through
the bodies those dummy links become — the import keeps them as links, on
purpose (ADR-0012), which is what the updated `import_urdf` snapshot shows
in the tree.

Both directories pass: 35 body and site poses each, to 1e-6, zero compiler
warnings.

snapshots: import_urdf gains the two imported dummy-link rows, which widens
the tree panel and moves the joint glyphs a few pixels.

File: assets/fixtures/arm/arm.urdf (robot description, URDF)
Before this commit: robot arm, 5 links, 4 joints
Links:
- added link camera_mount
- added link tcp
Joints:
- added joint camera_mount_fixed: type fixed, parent base, child camera_mount, origin xyz=0.03 0 0.015 rpy=0 1.570796326795 0
- added joint tcp_fixed: type fixed, parent fore, child tcp, origin xyz=0 0 0.08 rpy=0 0 0

Commit message: test(export,app): the arm carries a real mimic and MuJoCo agrees (plans/mimic-joints step 4)
`fore_joint` follows `upper_joint` at `-0.5 q + 0.1` in **both**
`arm.riggen` and `arm.urdf`, replacing the `multiplier="1" offset="0"` that
was only ever there to warn on. Neither coefficient is degenerate on
purpose: a multiplier of 1 and an offset of 0 would let a swapped
`polycoef` order pass unnoticed, which is the whole thing this step exists
to catch.

`test_mjcf_load.py` gains `check_equalities`: every `mjEQ_JOINT` must
reproduce the sampled `qpos` through its `polycoef`, and a pair of joints
the samples show as exactly coupled must have an equality — so both a
wrong coefficient order and a dropped `<equality>` fail. Verified both ways
by hand against the exported model.

The acceptance passes for both routes: `target/sample` and
`target/sample-urdf` load with no compiler warning, carry the equality, and
all 35 body and site poses match `riggen_core::fk` to 1e-6 at all five
configurations.

The offset means the forearm now sits at 0.1 rad even at rest, so the
sample's rest-pose numbers move with it.

snapshots: collision_hull, export_dialog, frame_properties, frames_tree and
import_urdf all show the same forearm, swung 0.1 rad about Y.

File: assets/fixtures/arm/arm.urdf (robot description, URDF)
Before this commit: robot arm, 7 links, 6 joints
Joints:
- joint fore_joint: mimic joint=upper_joint multiplier=1 offset=0 -> joint=upper_joint multiplier=-0.5 offset=0.1
